Commit message: max_trq_change

File: models/sample_bipedal_robot/sbr1.urdf (robot description, URDF)
Before this commit: robot sample_bipedal_robot, 13 links, 12 joints
Joints:
- joint ankle_pitch_left_joint: limit lower=-1.57 upper=1.57 effort=100 velocity=10 -> lower=-1.57 upper=1.57 effort=500 velocity=10
- joint ankle_pitch_right_joint: limit lower=-1.57 upper=1.57 effort=100 velocity=10 -> lower=-1.57 upper=1.57 effort=500 velocity=10
- joint ankle_roll_left_joint: limit lower=-1.57 upper=1.57 effort=100 velocity=10 -> lower=-1.57 upper=1.57 effort=500 velocity=10
- joint ankle_roll_right_joint: limit lower=-1.57 upper=1.57 effort=100 velocity=10 -> lower=-1.57 upper=1.57 effort=500 velocity=10
- joint hip_pitch_left_joint: limit lower=-1.57 upper=1.57 effort=100 velocity=10 -> lower=-1.57 upper=1.57 effort=500 velocity=10
- joint hip_pitch_right_joint: limit lower=-1.57 upper=1.57 effort=100 velocity=10 -> lower=-1.57 upper=1.57 effort=500 velocity=10
- joint hip_roll_right_joint: limit lower=-1.57 upper=1.57 effort=100 velocity=10 -> lower=-1.57 upper=1.57 effort=500 velocity=10
- joint hip_yaw_left_joint: limit lower=-1.57 upper=1.57 effort=100 velocity=10 -> lower=-1.57 upper=1.57 effort=500 velocity=10
- joint hip_yaw_right_joint: limit lower=-1.57 upper=1.57 effort=100 velocity=10 -> lower=-1.57 upper=1.57 effort=500 velocity=10
- joint knee_pitch_left_joint: limit lower=-1.57 upper=1.57 effort=100 velocity=10 -> lower=-1.57 upper=1.57 effort=500 velocity=10
- joint knee_pitch_right_joint: limit lower=-1.57 upper=1.57 effort=100 velocity=10 -> lower=-1.57 upper=1.57 effort=500 velocity=10
